Commit message: Fix pre-commit errors

File: src/yumi_config/config/moveit/yumi.ros2_control.xacro (robot description, xacro)
@@ -1,14 +1,13 @@
 <?xml version="1.0"?>
 <robot xmlns:xacro="http://www.ros.org/wiki/xacro">
-    <xacro:macro name="yumi_ros2_control" params="name initial_positions_file">
-        <xacro:property name="initial_positions" value="${xacro.load_yaml(initial_positions_file)['initial_positions']}"/>
-        <ros2_control name="yumi_control" type="system">
-            <hardware>
-            <!-- TODO: Pass in hardware_interface, scene_name, scene_package args
-              <xacro:if value="${hardware_interface == 'mock'}">
-                <plugin>mock_components/GenericSystem</plugin>
-                <param name="prefix">${prefix}</param>
-              </xacro:if>
-              <xacro:if value="${hardware_interface == 'sim'}">
+  <!-- Robot control -->
+  <xacro:macro name="yumi_ros2_control" params="name initial_positions_file hardware_interface">
+      <xacro:property name="initial_positions" value="${xacro.load_yaml(initial_positions_file)['initial_positions']}"/>
+      <ros2_control name="yumi_control" type="system">
+          <hardware>
+            <xacro:if value="${hardware_interface == 'mock'}">
+              <plugin>mock_components/GenericSystem</plugin>
+            </xacro:if>
+            <xacro:if value="${hardware_interface == 'sim'}">
               <plugin>picknik_mujoco_ros/MujocoSystem</plugin>
               <param name="mujoco_model">yumi_description/urdf/scene.xml</param>
@@ -17,5 +16,6 @@
               <param name="render_publish_rate">10</param>
               <param name="tf_publish_rate">60</param>
-               </xacro:if> -->
+            </xacro:if> -->
+            <xacro:if value="${hardware_interface == 'real'}">
               <plugin>abb_hardware_interface/ABBSystemHardware</plugin>
               <param name="rws_port">80</param>
@@ -23,134 +23,135 @@
               <!-- The following parameter is used for non-MultiMove only -->
               <param name="egm_port">6511</param>
-            </hardware>
-            <joint name="yumi_joint_1_l">
-                <command_interface name="position"/>
-                <state_interface name="position">
-                  <param name="initial_value">${initial_positions['yumi_joint_1_l']}</param>
-                </state_interface>
-                <state_interface name="velocity"/>
-                <state_interface name="effort"/>
-            </joint>
-            <joint name="yumi_joint_2_l">
-                <command_interface name="position"/>
-                <state_interface name="position">
-                  <param name="initial_value">${initial_positions['yumi_joint_2_l']}</param>
-                </state_interface>
-                <state_interface name="velocity"/>
-                <state_interface name="effort"/>
-            </joint>
-            <joint name="yumi_joint_7_l">
-                <command_interface name="position"/>
-                <state_interface name="position">
-                  <param name="initial_value">${initial_positions['yumi_joint_7_l']}</param>
-                </state_interface>
-                <state_interface name="velocity"/>
-                <state_interface name="effort"/>
-            </joint>
-            <joint name="yumi_joint_3_l">
-                <command_interface name="position"/>
-                <state_interface name="position">
-                  <param name="initial_value">${initial_positions['yumi_joint_3_l']}</param>
-                </state_interface>
-                <state_interface name="velocity"/>
-                <state_interface name="effort"/>
-            </joint>
-            <joint name="yumi_joint_4_l">
-                <command_interface name="position"/>
-                <state_interface name="position">
-                  <param name="initial_value">${initial_positions['yumi_joint_4_l']}</param>
-                </state_interface>
-                <state_interface name="velocity"/>
-                <state_interface name="effort"/>
-            </joint>
-            <joint name="yumi_joint_5_l">
-                <command_interface name="position"/>
-                <state_interface name="position">
-                  <param name="initial_value">${initial_positions['yumi_joint_5_l']}</param>
-                </state_interface>
-                <state_interface name="velocity"/>
-                <state_interface name="effort"/>
-            </joint>
-            <joint name="yumi_joint_6_l">
-                <command_interface name="position"/>
-                <state_interface name="position">
-                  <param name="initial_value">${initial_positions['yumi_joint_6_l']}</param>
-                </state_interface>
-                <state_interface name="velocity"/>
-                <state_interface name="effort"/>
-            </joint>
-            <joint name="yumi_joint_1_r">
-                <command_interface name="position"/>
-                <state_interface name="position">
-                  <param name="initial_value">${initial_positions['yumi_joint_1_r']}</param>
-                </state_interface>
-                <state_interface name="velocity"/>
-                <state_interface name="effort"/>
-            </joint>
-            <joint name="yumi_joint_2_r">
-                <command_interface name="position"/>
-                <state_interface name="position">
-                  <param name="initial_value">${initial_positions['yumi_joint_2_r']}</param>
-                </state_interface>
-                <state_interface name="velocity"/>
-                <state_interface name="effort"/>
-            </joint>
-            <joint name="yumi_joint_7_r">
-                <command_interface name="position"/>
-                <state_interface name="position">
-                  <param name="initial_value">${initial_positions['yumi_joint_7_r']}</param>
-                </state_interface>
-                <state_interface name="velocity"/>
-                <state_interface name="effort"/>
-            </joint>
-            <joint name="yumi_joint_3_r">
-                <command_interface name="position"/>
-                <state_interface name="position">
-                  <param name="initial_value">${initial_positions['yumi_joint_3_r']}</param>
-                </state_interface>
-                <state_interface name="velocity"/>
-                <state_interface name="effort"/>
-            </joint>
-            <joint name="yumi_joint_4_r">
-                <command_interface name="position"/>
-                <state_interface name="position">
-                  <param name="initial_value">${initial_positions['yumi_joint_4_r']}</param>
-                </state_interface>
-                <state_interface name="velocity"/>
-                <state_interface name="effort"/>
-            </joint>
-            <joint name="yumi_joint_5_r">
-                <command_interface name="position"/>
-                <state_interface name="position">
-                  <param name="initial_value">${initial_positions['yumi_joint_5_r']}</param>
-                </state_interface>
-                <state_interface name="velocity"/>
-                <state_interface name="effort"/>
-            </joint>
-            <joint name="yumi_joint_6_r">
-                <command_interface name="position"/>
-                <state_interface name="position">
-                  <param name="initial_value">${initial_positions['yumi_joint_6_r']}</param>
-                </state_interface>
-                <state_interface name="velocity"/>
-                <state_interface name="effort"/>
-            </joint>
-            <joint name="gripper_l_joint">
-                <command_interface name="position"/>
-                <state_interface name="position">
-                  <param name="initial_value">${initial_positions['gripper_l_joint']}</param>
-                </state_interface>
-                <state_interface name="velocity"/>
-                <state_interface name="effort"/>
-            </joint>
-            <joint name="gripper_r_joint">
-                <command_interface name="position"/>
-                <state_interface name="position">
-                  <param name="initial_value">${initial_positions['gripper_r_joint']}</param>
-                </state_interface>
-                <state_interface name="velocity"/>
-                <state_interface name="effort"/>
-            </joint>
-        </ros2_control>
-    </xacro:macro>
+            </xacro:if>
+          </hardware>
+          <joint name="yumi_joint_1_l">
+              <command_interface name="position"/>
+              <state_interface name="position">
+                <param name="initial_value">${initial_positions['yumi_joint_1_l']}</param>
+              </state_interface>
+              <state_interface name="velocity"/>
+              <state_interface name="effort"/>
+          </joint>
+          <joint name="yumi_joint_2_l">
+              <command_interface name="position"/>
+              <state_interface name="position">
+                <param name="initial_value">${initial_positions['yumi_joint_2_l']}</param>
+              </state_interface>
+              <state_interface name="velocity"/>
+              <state_interface name="effort"/>
+          </joint>
+          <joint name="yumi_joint_7_l">
+              <command_interface name="position"/>
+              <state_interface name="position">
+                <param name="initial_value">${initial_positions['yumi_joint_7_l']}</param>
+              </state_interface>
+              <state_interface name="velocity"/>
+              <state_interface name="effort"/>
+          </joint>
+          <joint name="yumi_joint_3_l">
+              <command_interface name="position"/>
+              <state_interface name="position">
+                <param name="initial_value">${initial_positions['yumi_joint_3_l']}</param>
+              </state_interface>
+              <state_interface name="velocity"/>
+              <state_interface name="effort"/>
+          </joint>
+          <joint name="yumi_joint_4_l">
+              <command_interface name="position"/>
+              <state_interface name="position">
+                <param name="initial_value">${initial_positions['yumi_joint_4_l']}</param>
+              </state_interface>
+              <state_interface name="velocity"/>
+              <state_interface name="effort"/>
+          </joint>
+          <joint name="yumi_joint_5_l">
+              <command_interface name="position"/>
+              <state_interface name="position">
+                <param name="initial_value">${initial_positions['yumi_joint_5_l']}</param>
+              </state_interface>
+              <state_interface name="velocity"/>
+              <state_interface name="effort"/>
+          </joint>
+          <joint name="yumi_joint_6_l">
+              <command_interface name="position"/>
+              <state_interface name="position">
+                <param name="initial_value">${initial_positions['yumi_joint_6_l']}</param>
+              </state_interface>
+              <state_interface name="velocity"/>
+              <state_interface name="effort"/>
+          </joint>
+          <joint name="yumi_joint_1_r">
+              <command_interface name="position"/>
+              <state_interface name="position">
+                <param name="initial_value">${initial_positions['yumi_joint_1_r']}</param>
+              </state_interface>
+              <state_interface name="velocity"/>
+              <state_interface name="effort"/>
+          </joint>
+          <joint name="yumi_joint_2_r">
+              <command_interface name="position"/>
+              <state_interface name="position">
+                <param name="initial_value">${initial_positions['yumi_joint_2_r']}</param>
+              </state_interface>
+              <state_interface name="velocity"/>
+              <state_interface name="effort"/>
+          </joint>
+          <joint name="yumi_joint_7_r">
+              <command_interface name="position"/>
+              <state_interface name="position">
+                <param name="initial_value">${initial_positions['yumi_joint_7_r']}</param>
+              </state_interface>
+              <state_interface name="velocity"/>
+              <state_interface name="effort"/>
+          </joint>
+          <joint name="yumi_joint_3_r">
+              <command_interface name="position"/>
+              <state_interface name="position">
+                <param name="initial_value">${initial_positions['yumi_joint_3_r']}</param>
+              </state_interface>
+              <state_interface name="velocity"/>
+              <state_interface name="effort"/>
+          </joint>
+          <joint name="yumi_joint_4_r">
+              <command_interface name="position"/>
+              <state_interface name="position">
+                <param name="initial_value">${initial_positions['yumi_joint_4_r']}</param>
+              </state_interface>
+              <state_interface name="velocity"/>
+              <state_interface name="effort"/>
+          </joint>
+          <joint name="yumi_joint_5_r">
+              <command_interface name="position"/>
+              <state_interface name="position">
+                <param name="initial_value">${initial_positions['yumi_joint_5_r']}</param>
+              </state_interface>
+              <state_interface name="velocity"/>
+              <state_interface name="effort"/>
+          </joint>
+          <joint name="yumi_joint_6_r">
+              <command_interface name="position"/>
+              <state_interface name="position">
+                <param name="initial_value">${initial_positions['yumi_joint_6_r']}</param>
+              </state_interface>
+              <state_interface name="velocity"/>
+              <state_interface name="effort"/>
+          </joint>
+          <joint name="gripper_l_joint">
+              <command_interface name="position"/>
+              <state_interface name="position">
+                <param name="initial_value">${initial_positions['gripper_l_joint']}</param>
+              </state_interface>
+              <state_interface name="velocity"/>
+              <state_interface name="effort"/>
+          </joint>
+          <joint name="gripper_r_joint">
+              <command_interface name="position"/>
+              <state_interface name="position">
+                <param name="initial_value">${initial_positions['gripper_r_joint']}</param>
+              </state_interface>
+              <state_interface name="velocity"/>
+              <state_interface name="effort"/>
+          </joint>
+      </ros2_control>
+  </xacro:macro>
 </robot>

File: src/yumi_config/config/moveit/yumi.urdf.xacro (robot description, xacro)
@@ -1,15 +1,21 @@
 <?xml version="1.0"?>
 <robot xmlns:xacro="http://www.ros.org/wiki/xacro" name="yumi">
-    <xacro:arg name="initial_positions_file" default="initial_positions.yaml" />
-    <!-- Import yumi urdf file -->
-    <xacro:include filename="$(find yumi_config)/yumi_description/urdf/yumi.urdf" />
-    <!-- Import control_xacro -->
-    <xacro:include filename="yumi.ros2_control.xacro" />
-    <link name="world"/>
-    <joint name="world_to_base" type="fixed">
-      <parent link="world"/>
-      <child link="yumi_base_link"/>
-      <origin xyz="0 0 0.25" rpy="0 0 1.57"/>
-    </joint>
-    <xacro:yumi_ros2_control name="FakeSystem" initial_positions_file="$(arg initial_positions_file)"/>
+  <xacro:arg name="initial_positions_file" default="initial_positions.yaml" />
+  <xacro:arg name="hardware_interface" default="mock"/>
+  <xacro:property name="hardware_interface" value="$(arg hardware_interface)"/>
+  <xacro:arg name="rws_ip" default="None"/>
+  <xacro:property name="rws_ip" value="$(arg rws_ip)"/>
+  <xacro:arg name="rws_port" default="80"/>
+  <xacro:property name="rws_port" value="$(arg rws_port)"/>
+  <!-- Import yumi urdf file -->
+  <xacro:include filename="$(find yumi_config)/yumi_description/urdf/yumi.urdf" />
+  <!-- Import control_xacro -->
+  <xacro:include filename="yumi.ros2_control.xacro" />
+  <link name="world"/>
+  <joint name="world_to_base" type="fixed">
+    <parent link="world"/>
+    <child link="yumi_base_link"/>
+    <origin xyz="0 0 0.25" rpy="0 0 1.57"/>
+  </joint>
+  <xacro:yumi_ros2_control name="YumiSystem" initial_positions_file="$(arg initial_positions_file)" hardware_interface="$(arg hardware_interface)"/>
 </robot>
